File: hw/lite/PiStackMon_lite.kicad_sch (KiCad schematic)
At the start: 31 parts, among them J1 Conn_01x03, J2 Conn_01x03, J3 5.08mm, J5 CUI PJ-102, P1 Conn_02x20_Odd_Even, U1 STP16CP05TTR

Commit message: Updating LED driver to TLC59282
Parts:
- R2: value 4k3 -> 10k; LCSC C23159 -> C25804
- U1: value STP16CP05TTR -> TLC59282DBQR; footprint Package_SO:TSSOP-24_4.4x7.8mm_P0.65mm -> Package_SO:SSOP-24_3.9x8.7mm_P0.635mm; JLC TSSOP-24_4.4x7.8x0.65P -> SSOP-24_3.9x8.7x0.635P; LCSC C127267 -> C129352
Changed lines of the file:
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@@
     (in_bom yes) (on_board yes)
     (property "Reference" "U1" (id 0) (at 198.12 111.76 0))
-    (property "Value" "STP16CP05TTR" (id 1) (at 200.66 114.3 0))
-    (property "Footprint" "Package_SO:TSSOP-24_4.4x7.8mm_P0.65mm" (id 2) (at 228.6 104.14 0)
-      (effects (font (size 1.27 1.27)) hide)
-    )
-    (property "Datasheet" "https://www.st.com/resource/en/datasheet/stp16cp05.pdf" (id 3) (at 228.6 104.14 0)
-      (effects (font (size 1.27 1.27)) hide)
-    )
-    (property "LCSC" "C127267" (id 4) (at 228.6 104.14 0)
-      (effects (font (size 1.27 1.27)) hide)
-    )
-    (property "JLC" "TSSOP-24_4.4x7.8x0.65P" (id 5) (at 228.6 104.14 0)
+    (property "Value" "TLC59282DBQR" (id 1) (at 200.66 114.3 0))
+    (property "Footprint" "Package_SO:SSOP-24_3.9x8.7mm_P0.635mm" (id 2) (at 228.6 104.14 0)
+      (effects (font (size 1.27 1.27)) hide)
+    )
+    (property "Datasheet" "https://datasheet.lcsc.com/lcsc/1809272034_Texas-Instruments-TLC59282DBQR_C129352.pdf" (id 3) (at 228.6 104.14 0)
+      (effects (font (size 1.27 1.27)) hide)
+    )
+    (property "LCSC" "C129352" (id 4) (at 228.6 104.14 0)
+      (effects (font (size 1.27 1.27)) hide)
+    )
+    (property "JLC" "SSOP-24_3.9x8.7x0.635P" (id 5) (at 228.6 104.14 0)
       (effects (font (size 1.27 1.27)) hide)
     )
@@
     (in_bom yes) (on_board yes)
     (property "Reference" "R2" (id 0) (at 213.36 123.19 90))
-    (property "Value" "4k3" (id 1) (at 218.44 123.19 90))
+    (property "Value" "10k" (id 1) (at 218.44 123.19 90))
     (property "Footprint" "Resistor_SMD:R_0603_1608Metric" (id 2) (at 214.122 123.19 90)
       (effects (font (size 1.27 1.27)) hide)
@@
       (effects (font (size 1.27 1.27)) hide)
     )
-    (property "LCSC" "C23159" (id 4) (at 215.9 123.19 0)
+    (property "LCSC" "C25804" (id 4) (at 215.9 123.19 0)
       (effects (font (size 1.27 1.27)) hide)
     )
@@
     )
     (path "/00000000-0000-0000-0000-000060137dbc"
-      (reference "R2") (unit 1) (value "4k3") (footprint "Resistor_SMD:R_0603_1608Metric")
+      (reference "R2") (unit 1) (value "10k") (footprint "Resistor_SMD:R_0603_1608Metric")
     )
     (path "/00000000-0000-0000-0000-00005ff5785f"
@@
     )
     (path "/00000000-0000-0000-0000-000060133f70"
-      (reference "U1") (unit 1) (value "STP16CP05TTR") (footprint "Package_SO:TSSOP-24_4.4x7.8mm_P0.65mm")
-    )
-  )
+      (reference "U1") (unit 1) (value "TLC59282DBQR") (footprint "Package_SO:SSOP-24_3.9x8.7mm_P0.635mm")
+    )
+  )

Commit message: Minor changes based on @bablokb's feedback
Parts:
- added C2: 100n, Capacitor_SMD:C_0402_1005Metric, symbol Device:C_Small
- added R1, R4: NM, Resistor_SMD:R_0805_2012Metric_Pad1.20x1.40mm_HandSolder, symbol Device:R
- added R5: 3k3, Resistor_SMD:R_0402_1005Metric, symbol Device:R
- R3: value 1k -> 560R; LCSC C21190 -> C23204
Connections:
- net +3V3: now also C2.1, R5.2
- net 3V3_2: now also J1.3 (Pin_3), R1.1, R4.1
- net GND: now also C2.2; no longer U1.21 (~{OE/DM2})
- net GPIO2(SDA1): now also J1.1 (Pin_1), R4.2; no longer J1.3 (Pin_3)
- net GPIO25(GEN6): now also U1.21 (~{OE/DM2}), R5.1
- net GPIO3(SCL1): now also R1.2
- net GPIO4(1Wire_Default): no longer J1.1 (Pin_1)
Other:
- note added: "Optional I2C Pullups"
- moved on the sheet: J1, J2, R2

Commit message: Resistor values tweak (LEDs were too bright)
Parts:
- R2: value 10k -> 27k; LCSC C25804 -> C22967
- R3: value 560R -> 1k8; LCSC C23204 -> C4177
Changed lines of the file:
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@@
       (effects (font (size 1.27 1.27)) (justify left))
     )
-    (property "Value" "560R" (id 1) (at 271.018 138.303 0)
+    (property "Value" "1k8" (id 1) (at 271.018 138.303 0)
       (effects (font (size 1.27 1.27)) (justify left))
     )
@@
       (effects (font (size 1.27 1.27)) hide)
     )
-    (property "LCSC" "C23204" (id 4) (at 269.24 137.16 0)
+    (property "LCSC" "C4177" (id 4) (at 269.24 137.16 0)
       (effects (font (size 1.27 1.27)) hide)
     )
@@
     (in_bom yes) (on_board yes)
     (property "Reference" "R2" (id 0) (at 213.36 119.38 90))
-    (property "Value" "10k" (id 1) (at 218.44 119.38 90))
+    (property "Value" "27k" (id 1) (at 218.44 119.38 90))
     (property "Footprint" "Resistor_SMD:R_0603_1608Metric" (id 2) (at 214.122 119.38 90)
       (effects (font (size 1.27 1.27)) hide)
@@
       (effects (font (size 1.27 1.27)) hide)
     )
-    (property "LCSC" "C25804" (id 4) (at 215.9 119.38 0)
+    (property "LCSC" "C22967" (id 4) (at 215.9 119.38 0)
       (effects (font (size 1.27 1.27)) hide)
     )
@@
     )
     (path "/00000000-0000-0000-0000-000060137dbc"
-      (reference "R2") (unit 1) (value "10k") (footprint "Resistor_SMD:R_0603_1608Metric")
+      (reference "R2") (unit 1) (value "27k") (footprint "Resistor_SMD:R_0603_1608Metric")
     )
     (path "/00000000-0000-0000-0000-00005ff5785f"
-      (reference "R3") (unit 1) (value "560R") (footprint "Resistor_SMD:R_0603_1608Metric")
+      (reference "R3") (unit 1) (value "1k8") (footprint "Resistor_SMD:R_0603_1608Metric")
     )
     (path "/356a997d-9f21-4014-b1ae-7da6a8302796"
